Commit message: 6.28

File: work_ws/src/kai01_description/urdf/arm.urdf.xacro (robot description, xacro)
@@ -2,4 +2,16 @@
 <robot name="arm" xmlns:xacro="http://ros.org/wiki/xacro">
   <xacro:property name="M_PI"   value="3.1415926535897931"/>
+  <link name="gripper_tcp"> </link>
+  <joint
+    name="gripper_tcp_coupling"
+    type="fixed">
+    <origin
+      xyz="0 0 0.117"
+      rpy="0 0 0" />
+    <parent
+      link="coupling" />
+    <child
+      link="gripper_tcp" />
+  </joint>
   <link
     name="arm_base_link"> <!-- 机械臂底座 -->

File: work_ws/src/kai01_description/urdf/car_mecanum.urdf.xacro (robot description, xacro)
@@ -11,5 +11,11 @@
     <parent link="base_footprint"/>
     <child link="base_link"/>
-    <origin xyz="0.0 0.0 ${0.0965/2 + 0.0678410821576746}" rpy="0 0 0"/>
+    <origin xyz="0.0 0.0 0.12" rpy="0 0 0"/>
+  </joint>
+  <link name="measure"/><!-- 测量点 -->
+  <joint name="measure_joint" type="fixed">
+    <parent link="base_footprint"/>
+    <child link="measure"/>
+    <origin xyz="0.153 0.0 0.0" rpy="0 0 0"/>
   </joint>
   <link
