Commit message: 7.17

File: work_ws/src/kai01_description/urdf/car_mecanum.urdf.xacro (robot description, xacro)
@@ -15,7 +15,7 @@
   <link name="measure"/><!-- 测量点 -->
   <joint name="measure_joint" type="fixed">
-    <parent link="base_footprint"/>
-    <child link="measure"/>
-    <origin xyz="0.153 0.0 0.0" rpy="0 0 0"/>
+    <parent link="measure"/>
+    <child link="base_footprint"/>
+    <origin xyz="-0.153 0.0 0.0" rpy="0 0 0"/>
   </joint>
   <link

Commit message: 修复重定位问题

File: work_ws/src/kai01_description/urdf/car_mecanum.urdf.xacro (robot description, xacro)
@@ -13,10 +13,4 @@
     <origin xyz="0.0 0.0 0.12" rpy="0 0 0"/>
   </joint>
-  <link name="measure"/><!-- 测量点 -->
-  <joint name="measure_joint" type="fixed">
-    <parent link="measure"/>
-    <child link="base_footprint"/>
-    <origin xyz="-0.153 0.0 0.0" rpy="0 0 0"/>
-  </joint>
   <link
     name="base_link"> <!-- 下底盘 -->
